File: AJH_as3340_VCO/AJH_as3340_20.sch (EAGLE design)
At the start: 98 parts, among them IC1 LM4040 5.0V, IC2 TL072D, IC3 TL072D, IC4 TL072D, IC5 CEM3340SOIC16, IC6 TL072D, IC7 TL072D

Commit message: Arranged UI
Parts:
- JP2: value M05X2SMD -> (none); device og-header:M05X2SMD -> jumper:JP5Q
Changed lines of the file:
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@@
 </variantdefs>
 <classes>
-<class number="0" name="default" width="0" drill="0">
+<class number="0" name="default" width="0.2032" drill="0.2032">
+<clearance class="0" value="0.2032"/>
 </class>
-<class number="1" name="power" width="0.1778" drill="0.3048">
-<clearance class="0" value="0.1778"/>
-<clearance class="1" value="0.1778"/>
+<class number="1" name="power" width="0.3048" drill="0.3048">
+<clearance class="0" value="0.3048"/>
+<clearance class="1" value="0.3048"/>
 </class>
 </classes>
@@
 <part name="R6" library="resistor" deviceset="R-US_" device="R0603" value="100k"/>
 <part name="GND4" library="SparkFun" deviceset="GND" device=""/>
-<part name="JP2" library="og-header" deviceset="M05X2" device="SMD"/>
+<part name="JP2" library="jumper" library_urn="urn:adsk.eagle:library:252" deviceset="JP5Q" device="" package3d_urn="urn:adsk.eagle:package:15454/1"/>
 </parts>
 <sheets>
@@
 <instance part="D2" gate="G$1" x="-157.48" y="-116.84" smashed="yes">
 <attribute name="NAME" x="-154.94" y="-116.3574" size="1.778" layer="95"/>
-<attribute name="VALUE" x="-170.18" y="-124.2314" size="1.778" layer="96"/>
+<attribute name="VALUE" x="-167.64" y="-121.6914" size="1.778" layer="96"/>
 </instance>
 <instance part="D1" gate="G$1" x="-157.48" y="-106.68" smashed="yes" rot="R180">
@@
 <attribute name="VALUE" x="276.86" y="91.44" size="1.778" layer="96"/>
 </instance>
-<instance part="JP2" gate="G$1" x="-142.24" y="-111.76" smashed="yes" rot="MR180">
-<attribute name="VALUE" x="-144.78" y="-101.6" size="1.778" layer="96" rot="MR180"/>
-<attribute name="NAME" x="-144.78" y="-120.142" size="1.778" layer="95" rot="MR180"/>
+<instance part="JP2" gate="B" x="-142.24" y="-111.76" smashed="yes" rot="MR90">
+<attribute name="VALUE" x="-152.4" y="-114.3" size="1.778" layer="96" rot="MR90"/>
+<attribute name="NAME" x="-147.32" y="-120.142" size="1.778" layer="95" rot="MR180"/>
 </instance>
 </instances>
@@
 <wire x1="-132.08" y1="-114.3" x2="-132.08" y2="-116.84" width="0.1524" layer="91"/>
 <pinref part="GND11" gate="1" pin="GND"/>
-<pinref part="JP2" gate="G$1" pin="4"/>
-<pinref part="JP2" gate="G$1" pin="8"/>
-<pinref part="JP2" gate="G$1" pin="6"/>
+<pinref part="JP2" gate="B" pin="4"/>
+<pinref part="JP2" gate="B" pin="8"/>
+<pinref part="JP2" gate="B" pin="6"/>
 <wire x1="-134.62" y1="-109.22" x2="-134.62" y2="-111.76" width="0.1524" layer="91"/>
 <wire x1="-134.62" y1="-114.3" x2="-134.62" y2="-111.76" width="0.1524" layer="91"/>
 <junction x="-134.62" y="-114.3"/>
 <junction x="-134.62" y="-111.76"/>
-<pinref part="JP2" gate="G$1" pin="7"/>
-<pinref part="JP2" gate="G$1" pin="5"/>
+<pinref part="JP2" gate="B" pin="7"/>
+<pinref part="JP2" gate="B" pin="5"/>
 <wire x1="-149.86" y1="-109.22" x2="-149.86" y2="-111.76" width="0.1524" layer="91"/>
-<pinref part="JP2" gate="G$1" pin="3"/>
+<pinref part="JP2" gate="B" pin="3"/>
 <wire x1="-149.86" y1="-111.76" x2="-149.86" y2="-114.3" width="0.1524" layer="91"/>
 <junction x="-149.86" y="-111.76"/>
@@
 <pinref part="D1" gate="G$1" pin="A"/>
 <wire x1="-149.86" y1="-106.68" x2="-154.94" y2="-106.68" width="0.1524" layer="91"/>
-<pinref part="JP2" gate="G$1" pin="9"/>
-<pinref part="JP2" gate="G$1" pin="10"/>
+<pinref part="JP2" gate="B" pin="9"/>
+<pinref part="JP2" gate="B" pin="10"/>
 <wire x1="-134.62" y1="-106.68" x2="-149.86" y2="-106.68" width="0.1524" layer="91"/>
 <junction x="-149.86" y="-106.68"/>
@@
 <pinref part="D2" gate="G$1" pin="C"/>
 <wire x1="-149.86" y1="-116.84" x2="-154.94" y2="-116.84" width="0.1524" layer="91"/>
-<pinref part="JP2" gate="G$1" pin="1"/>
-<pinref part="JP2" gate="G$1" pin="2"/>
+<pinref part="JP2" gate="B" pin="1"/>
+<pinref part="JP2" gate="B" pin="2"/>
 <wire x1="-134.62" y1="-116.84" x2="-149.86" y2="-116.84" width="0.1524" layer="91"/>
 <junction x="-149.86" y="-116.84"/>
